File: pcb/pcb_pcBOT/bms.kicad_sch (KiCad schematic)
At the start: 1 part, among them U1 BQ25895RTW

Commit message: pcb
Parts:
- removed U1: BQ25895RTW, Package_DFN_QFN:Texas_S-PWQFN-N24_EP2.7x2.7mm_ThermalVias, symbol Battery_Management:BQ25895RTW
Other:
- title: BMS BQ25896RTWR -> (none)
Changed lines of the file:
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@@
 (kicad_sch (version 20230121) (generator eeschema)
   (paper "A4")
-  (title_block
-    (title "BMS BQ25896RTWR")
-    (rev "1.0")
-  )
-  (symbol (lib_id "Battery_Management:BQ25895RTW") (at 116.84 106.68 0) (unit 1)
-    (in_bom yes) (on_board yes) (dnp no) (fields_autoplaced)
-    (property "Reference" "U1" (at 116.84 82.55 0)
-      (effects (font (size 1.27 1.27)))
-    )
-    (property "Value" "BQ25895RTW" (at 116.84 85.09 0)
-      (effects (font (size 1.27 1.27)))
-    )
-    (property "Footprint" "Package_DFN_QFN:Texas_S-PWQFN-N24_EP2.7x2.7mm_ThermalVias" (at 114.3 81.28 0)
-      (effects (font (size 1.27 1.27)) hide)
-    )
-    (property "Datasheet" "http://www.ti.com/lit/ds/symlink/bq25895.pdf" (at 111.76 86.36 0)
-      (effects (font (size 1.27 1.27)) hide)
-    )
-    (pin "1")
-    (pin "10")
-    (pin "11")
-    (pin "12")
-    (pin "13")
-    (pin "14")
-    (pin "15")
-    (pin "16")
-    (pin "17")
-    (pin "18")
-    (pin "19")
-    (pin "2")
-    (pin "20")
-    (pin "21")
-    (pin "22")
-    (pin "23")
-    (pin "24")
-    (pin "25")
-    (pin "3")
-    (pin "4")
-    (pin "5")
-    (pin "6")
-    (pin "7")
-    (pin "8")
-    (pin "9")
-    (instances
-      (project "pcb_pcBOT"
-        (path "/704e4da3-8ee7-458f-8a0f-3fc97e8dc2a6/d67675e6-7dac-4bc7-9bdf-0364d005735e"
-          (reference "U1") (unit 1)
-        )
-      )
-    )
-  )
 )

Commit message: ajout de la librairie composant
Parts:
- added U1: BQ25895RTW, Package_DFN_QFN:Texas_S-PWQFN-N24_EP2.7x2.7mm_ThermalVias, symbol Battery_Management:BQ25895RTW
Connections:
- new net: U1.13 (BAT), U1.14 (BAT)
- new net: U1.15 (SYS), U1.16 (SYS)
- new net: U1.17 (PGND), U1.18 (PGND), U1.25 (PGND)
- new net: U1.19 (SW), U1.20 (SW)
Other:
- title: (none) -> BMS BQ25896RTWR
Changed lines of the file:
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@@
 (kicad_sch (version 20230121) (generator eeschema)
   (paper "A4")
+  (title_block
+    (title "BMS BQ25896RTWR")
+    (rev "1.0")
+  )
+  (symbol (lib_id "Battery_Management:BQ25895RTW") (at 116.84 106.68 0) (unit 1)
+    (in_bom yes) (on_board yes) (dnp no) (fields_autoplaced)
+    (property "Reference" "U1" (at 116.84 82.55 0)
+      (effects (font (size 1.27 1.27)))
+    )
+    (property "Value" "BQ25895RTW" (at 116.84 85.09 0)
+      (effects (font (size 1.27 1.27)))
+    )
+    (property "Footprint" "Package_DFN_QFN:Texas_S-PWQFN-N24_EP2.7x2.7mm_ThermalVias" (at 114.3 81.28 0)
+      (effects (font (size 1.27 1.27)) hide)
+    )
+    (property "Datasheet" "http://www.ti.com/lit/ds/symlink/bq25895.pdf" (at 111.76 86.36 0)
+      (effects (font (size 1.27 1.27)) hide)
+    )
+    (pin "1")
+    (pin "10")
+    (pin "11")
+    (pin "12")
+    (pin "13")
+    (pin "14")
+    (pin "15")
+    (pin "16")
+    (pin "17")
+    (pin "18")
+    (pin "19")
+    (pin "2")
+    (pin "20")
+    (pin "21")
+    (pin "22")
+    (pin "23")
+    (pin "24")
+    (pin "25")
+    (pin "3")
+    (pin "4")
+    (pin "5")
+    (pin "6")
+    (pin "7")
+    (pin "8")
+    (pin "9")
+    (instances
+      (project "pcb_pcBOT"
+        (path "/704e4da3-8ee7-458f-8a0f-3fc97e8dc2a6/d67675e6-7dac-4bc7-9bdf-0364d005735e"
+          (reference "U1") (unit 1)
+        )
+      )
+    )
+  )
 )
