File: pcb/pcb_pcBOT/bms.kicad_sch (KiCad schematic)
At the start: 20 parts, among them J201 Lipo, U201 BQ25896RTW

Commit message: update bms
Connections:
- net SCL_I2C is gone; now on net I2C_SCL: R203.2
- net SDA_I2C is gone; now on net I2C_SDA: R201.2
- net SYS is gone; now on net +5V: D201.2 (A), D202.2 (A)
- net SYS_3.5-4.5V is gone; now on net +5V: C205.1, C207.1, L201.2, U201.15 (SYS), U201.16 (SYS)
- net USB is gone; now on net VBUS: C201.1, U201.1 (VBUS)
- net SW: now reaches C203.1, L201.1, U201.19 (SW), U201.20 (SW)
- net BTST: now reaches C203.2, U201.21 (BTST)
- net BAT: now reaches C206.1, J201.1 (Pin_1), U201.13 (BAT), U201.14 (BAT)
- net TS: now reaches R207.2, R208.1, U201.11 (TS)
- net ILIM: now reaches R206.2, U201.10 (ILIM)
- net I2C_SCL: now reaches U201.5 (SCL)
- net VREF renamed +3.3V
- no-connect marks 1 -> 0
Other:
- moved on the sheet: R206

Commit message: fin bms schematic bms
Parts:
- added JP201, JP202, JP203: SolderJumper_2_Open, Jumper:SolderJumper-2_P1.3mm_Open_TrianglePad1.0x1.5mm, symbol Jumper:SolderJumper_2_Open
Connections:
- net +5V: now also JP202.2 (B); no longer C205.1, C207.1, D201.2 (A), D202.2 (A), L201.2, U201.15 (SYS), U201.16 (SYS)
- net VBUS: now also JP201.1 (A), JP203.1 (A); no longer U201.1 (VBUS)
- net PHY: no longer names the net of U201.2 (PSEL)
- net PHY: now also JP203.2 (B)
- new net: JP201.2 (B), U201.1 (VBUS)
- new net SYS: C205.1, C207.1, D201.2 (A), D202.2 (A), JP202.1 (A), L201.2, U201.15 (SYS), U201.16 (SYS)
Other:
- moved on the sheet: C204
