File: pcb/pcb_pcBOT/drv.kicad_sch (KiCad schematic)
At the start: 0 parts

Commit message: pcb
Parts:
- added M1: Stepper_Motor_bipolar, symbol Motor:Stepper_Motor_bipolar
- added R-IPROPI_A, R-IPROPI_B: R, symbol Device:R
- added U2: DRV8411A, Package_SO:HTSSOP-16-1EP_4.4x5mm_P0.65mm_EP3.4x5mm_Mask2.46x2.31mm_ThermalVias, symbol pcbot_lib:DRV8411A
Connections:
- new net: R-IPROPI_B.1, U2.11 (BIPROPI)
- new net: R-IPROPI_A.1, U2.14 (AIPROPI)
- new net: M1.2 (-), U2.2 (AOUT1)
- new net: M1.1, U2.4 (AOUT2)
- new net: M1.4, U2.5 (BOUT2)
- new net: M1.3, U2.7 (BOUT1)
- new net GND: R-IPROPI_A.2, R-IPROPI_B.2, U2.13 (GND), U2.17 (PPAD), U2.3 (PGNDA), U2.6 (PGNDB)
