File: pcb/pcb_pcBOT/drv.kicad_sch (KiCad schematic)
At the start: 8 parts, among them U701 DRV8411A

Commit message: modifs
Parts:
- removed Cbulk1: 10µF, symbol Device:C
- added C2: 100u, Capacitor_SMD:CP_Elec_6.3x3, symbol Device:C_Polarized_Small
- C1: footprint (none) -> Capacitor_SMD:C_0402_1005Metric
- Moteur1, Moteur2: footprint (none) -> Connector_PinSocket_2.54mm:PinSocket_1x02_P2.54mm_Vertical
- R-IPROPI_A1, R-IPROPI_B1, Rvmcu1: footprint (none) -> Resistor_SMD:R_0402_1005Metric
- U1: renamed from U701; footprint Package_SO:HTSSOP-16-1EP_4.4x5mm_P0.65mm_EP3.4x5mm_Mask2.46x2.31mm_ThermalVias -> Package_SO:HTSSOP-16-1EP_4.4x5mm_P0.65mm_EP3.4x5mm_Mask2.46x2.31mm
Connections:
- net +5V: now also C2.1
- net GND: now also C2.2
Changed lines of the file:
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@@
+	(wire
+		(pts
+			(xy 173.99 86.36) (xy 173.99 88.9)
+		)
+		(stroke
+			(width 0)
+			(type default)
+		)
+	)
 	(wire
 		(pts
@@
 				(justify right)
 				(hide yes)
-			)
-		)
-	)
-	(symbol
-		(lib_id "Device:C")
-		(at 173.99 85.09 0)
-		(unit 1)
-		(exclude_from_sim no)
-		(in_bom yes)
-		(on_board yes)
-		(dnp no)
-		(fields_autoplaced yes)
-		(property "Reference" "Cbulk1"
-			(at 177.8 83.8199 0)
-			(effects
-				(font
-					(size 1.27 1.27)
-				)
-				(justify left)
-			)
-		)
-		(property "Value" "10µF"
-			(at 177.8 86.3599 0)
-			(effects
-				(font
-					(size 1.27 1.27)
-				)
-				(justify left)
-			)
-		)
-		(property "Footprint" ""
-			(at 174.9552 88.9 0)
-			(effects
-				(font
-					(size 1.27 1.27)
-				)
-				(hide yes)
-			)
-		)
-		(property "Datasheet" "~"
-			(at 173.99 85.09 0)
-			(effects
-				(font
-					(size 1.27 1.27)
-				)
-				(hide yes)
-			)
-		)
-		(property "Description" "Unpolarized capacitor"
-			(at 173.99 85.09 0)
-			(effects
-				(font
-					(size 1.27 1.27)
-				)
-				(hide yes)
-			)
-		)
-		(pin "2"
-		)
-		(pin "1"
-		)
-		(instances
-			(project ""
-				(path "/704e4da3-8ee7-458f-8a0f-3fc97e8dc2a6/9be667e2-7a7b-40ab-9f7b-a44803d38fe0"
-					(reference "Cbulk1")
-					(unit 1)
-				)
 			)
 		)
@@
 		(on_board yes)
 		(dnp no)
-		(property "Reference" "U701"
+		(property "Reference" "U1"
 			(at 148.082 98.298 0)
 			(effects
@@
 			)
 		)
-		(property "Footprint" "Package_SO:HTSSOP-16-1EP_4.4x5mm_P0.65mm_EP3.4x5mm_Mask2.46x2.31mm_ThermalVias"
+		(property "Footprint" "Package_SO:HTSSOP-16-1EP_4.4x5mm_P0.65mm_EP3.4x5mm_Mask2.46x2.31mm"
 			(at 117.602 154.686 0)
 			(effects
@@
 		(dnp no)
 		(fields_autoplaced yes)
-		(property "Reference" "#PWR04"
+		(property "Reference" "#PWR01"
 			(at 119.38 101.6 0)
 			(effects
@@
 		)
 		(instances
+			(project "drv"
+				(path "/2fd91a2b-5865-4ecc-b351-728089a193d5"
+					(reference "#PWR01")
+					(unit 1)
+				)
+			)
 			(project ""
 				(path "/704e4da3-8ee7-458f-8a0f-3fc97e8dc2a6/9be667e2-7a7b-40ab-9f7b-a44803d38fe0"
@@
 			)
 		)
-		(property "Footprint" ""
+		(property "Footprint" "Resistor_SMD:R_0402_1005Metric"
 			(at 193.04 132.08 0)
 			(effects
@@
 					(size 1.27 1.27)
 				)
+				(hide yes)
 			)
 		)
@@
 			(project "drv"
 				(path "/2fd91a2b-5865-4ecc-b351-728089a193d5"
-					(reference "R-IPROPI_A")
+					(reference "R-IPROPI_A1")
 					(unit 1)
 				)
@@
 			)
 		)
-		(property "Footprint" ""
+		(property "Footprint" "Connector_PinSocket_2.54mm:PinSocket_1x02_P2.54mm_Vertical"
 			(at 170.18 113.03 0)
 			(effects
@@
 		)
 		(instances
+			(project "drv"
+				(path "/2fd91a2b-5865-4ecc-b351-728089a193d5"
+					(reference "Moteur2")
+					(unit 1)
+				)
+			)
 			(project "pcb_pcBOT"
 				(path "/704e4da3-8ee7-458f-8a0f-3fc97e8dc2a6/9be667e2-7a7b-40ab-9f7b-a44803d38fe0"
@@
 			)
 		)
-		(property "Footprint" ""
+		(property "Footprint" "Resistor_SMD:R_0402_1005Metric"
 			(at 181.61 132.08 0)
 			(effects
@@
 			(project "drv"
 				(path "/2fd91a2b-5865-4ecc-b351-728089a193d5"
-					(reference "R-IPROPI_B")
+					(reference "R-IPROPI_B1")
 					(unit 1)
 				)
@@
 		(on_board yes)
 		(dnp no)
-		(property "Reference" "#PWR0702"
+		(property "Reference" "#PWR05"
 			(at 168.91 138.43 0)
 			(effects
@@
 			(project "drv"
 				(path "/2fd91a2b-5865-4ecc-b351-728089a193d5"
-					(reference "#PWR?")
+					(reference "#PWR05")
 					(unit 1)
 				)
@@
 			)
 		)
-		(property "Footprint" ""
+		(property "Footprint" "Resistor_SMD:R_0402_1005Metric"
 			(at 119.38 119.38 0)
 			(effects
@@
 					(size 1.27 1.27)
 				)
+				(hide yes)
 			)
 		)
@@
 		)
 		(instances
+			(project "drv"
+				(path "/2fd91a2b-5865-4ecc-b351-728089a193d5"
+					(reference "Rvmcu1")
+					(unit 1)
+				)
+			)
 			(project "pcb_pcBOT"
 				(path "/704e4da3-8ee7-458f-8a0f-3fc97e8dc2a6/9be667e2-7a7b-40ab-9f7b-a44803d38fe0"
@@
 		(dnp no)
 		(fields_autoplaced yes)
-		(property "Reference" "#PWR0701"
+		(property "Reference" "#PWR03"
 			(at 146.05 148.59 0)
 			(effects
@@
 			(project "drv"
 				(path "/2fd91a2b-5865-4ecc-b351-728089a193d5"
-					(reference "#PWR?")
+					(reference "#PWR03")
 					(unit 1)
 				)
@@
 			)
 		)
-		(property "Footprint" ""
+		(property "Footprint" "Capacitor_SMD:C_0402_1005Metric"
 			(at 160.3248 81.28 0)
 			(effects
@@
 		)
 		(instances
+			(project "drv"
+				(path "/2fd91a2b-5865-4ecc-b351-728089a193d5"
+					(reference "C1")
+					(unit 1)
+				)
+			)
 			(project ""
 				(path "/704e4da3-8ee7-458f-8a0f-3fc97e8dc2a6/9be667e2-7a7b-40ab-9f7b-a44803d38fe0"
@@
 		(on_board yes)
 		(dnp no)
-		(property "Reference" "#PWR01"
+		(property "Reference" "#PWR04"
 			(at 161.29 95.25 0)
 			(effects
@@
 		)
 		(instances
+			(project "drv"
+				(path "/2fd91a2b-5865-4ecc-b351-728089a193d5"
+					(reference "#PWR04")
+					(unit 1)
+				)
+			)
 			(project "pcb_pcBOT"
 				(path "/704e4da3-8ee7-458f-8a0f-3fc97e8dc2a6/9be667e2-7a7b-40ab-9f7b-a44803d38fe0"
@@
 		(on_board yes)
 		(dnp no)
-		(property "Reference" "#PWR0703"
+		(property "Reference" "#PWR07"
 			(at 181.61 142.24 0)
 			(effects
@@
 			(project "drv"
 				(path "/2fd91a2b-5865-4ecc-b351-728089a193d5"
-					(reference "#PWR?")
+					(reference "#PWR07")
 					(unit 1)
 				)
@@
 			)
 		)
-		(property "Footprint" ""
+		(property "Footprint" "Connector_PinSocket_2.54mm:PinSocket_1x02_P2.54mm_Vertical"
 			(at 170.18 100.33 0)
 			(effects
@@
 		)
 		(instances
+			(project "drv"
+				(path "/2fd91a2b-5865-4ecc-b351-728089a193d5"
+					(reference "Moteur1")
+					(unit 1)
+				)
+			)
 			(project ""
 				(path "/704e4da3-8ee7-458f-8a0f-3fc97e8dc2a6/9be667e2-7a7b-40ab-9f7b-a44803d38fe0"
@@
 		(on_board yes)
 		(dnp no)
-		(property "Reference" "#PWR0704"
+		(property "Reference" "#PWR08"
 			(at 193.04 142.24 0)
 			(effects
@@
 			(project "drv"
 				(path "/2fd91a2b-5865-4ecc-b351-728089a193d5"
-					(reference "#PWR?")
+					(reference "#PWR08")
 					(unit 1)
 				)
@@
 				(path "/704e4da3-8ee7-458f-8a0f-3fc97e8dc2a6/9be667e2-7a7b-40ab-9f7b-a44803d38fe0"
 					(reference "#PWR0704")
+					(unit 1)
+				)
+			)
+		)
+	)
+	(symbol
+		(lib_id "Device:C_Polarized_Small")
+		(at 173.99 83.82 0)
+		(unit 1)
+		(exclude_from_sim no)
+		(in_bom yes)
+		(on_board yes)
+		(dnp no)
+		(fields_autoplaced yes)
+		(property "Reference" "C2"
+			(at 176.53 82.0038 0)
+			(effects
+				(font
+					(size 1.27 1.27)
+				)
+				(justify left)
+			)
+		)
+		(property "Value" "100u"
+			(at 176.53 84.5438 0)
+			(effects
+				(font
+					(size 1.27 1.27)
+				)
+				(justify left)
+			)
+		)
+		(property "Footprint" "Capacitor_SMD:CP_Elec_6.3x3"
+			(at 173.99 83.82 0)
+			(effects
+				(font
+					(size 1.27 1.27)
+				)
+				(hide yes)
+			)
+		)
+		(property "Datasheet" "~"
+			(at 173.99 83.82 0)
+			(effects
+				(font
+					(size 1.27 1.27)
+				)
+				(hide yes)
+			)
+		)
+		(property "Description" "Polarized capacitor, small symbol"
+			(at 173.99 83.82 0)
+			(effects
+				(font
+					(size 1.27 1.27)
+				)
+				(hide yes)
+			)
+		)
+		(pin "1"
+		)
+		(pin "2"
+		)
+		(instances
+			(project ""
+				(path "/2fd91a2b-5865-4ecc-b351-728089a193d5"
+					(reference "C2")
 					(unit 1)
 				)
@@
 		(on_board yes)
 		(dnp no)
-		(property "Reference" "#PWR02"
+		(property "Reference" "#PWR06"
 			(at 173.99 95.25 0)
 			(effects
@@
 		)
 		(instances
+			(project "drv"
+				(path "/2fd91a2b-5865-4ecc-b351-728089a193d5"
+					(reference "#PWR06")
+					(unit 1)
+				)
+			)
 			(project "pcb_pcBOT"
 				(path "/704e4da3-8ee7-458f-8a0f-3fc97e8dc2a6/9be667e2-7a7b-40ab-9f7b-a44803d38fe0"
@@
 		(dnp no)
 		(fields_autoplaced yes)
-		(property "Reference" "#PWR03"
+		(property "Reference" "#PWR02"
 			(at 146.05 80.01 0)
 			(effects
@@
 		)
 		(instances
+			(project "drv"
+				(path "/2fd91a2b-5865-4ecc-b351-728089a193d5"
+					(reference "#PWR02")
+					(unit 1)
+				)
+			)
 			(project ""
 				(path "/704e4da3-8ee7-458f-8a0f-3fc97e8dc2a6/9be667e2-7a7b-40ab-9f7b-a44803d38fe0"
