File: pcb/pcb_pcBOT/tof.kicad_sch (KiCad schematic)
At the start: 0 parts

Commit message: Description de mes changements
Parts:
- added 4,7: 100 nF, symbol Device:C
- added C1: C, symbol Device:C
- added U1: VL53L0CXV0DH1, Sensor_Distance:ST_VL53L1x, symbol Sensor_Distance:VL53L0CXV0DH1
Connections:
- new net: 4,7.1, C1.1, U1.1 (AVDDVCSEL), U1.11 (AVDD)
- new net: 4,7.2, C1.2, U1.12 (GND), U1.2 (AVSSVCSEL), U1.3 (GND), U1.4 (GND), U1.6 (GND)

Commit message: DRV fini
Parts:
- removed 4,7: 100 nF, symbol Device:C
- removed C1: C, symbol Device:C
- removed U1: VL53L0CXV0DH1, Sensor_Distance:ST_VL53L1x, symbol Sensor_Distance:VL53L0CXV0DH1
