File: pcb/pcb_pcBOT/stm32.kicad_sch (KiCad schematic)
At the start: 18 parts, among them J302 Conn_ST_STDC14, SW301 Reset_Button, U301 STM32G431KBT6, U303 BU33??

Commit message: rouatage + firmware wip
Parts:
- C301, C302, C303, C304, C305, C306, C307, C309: footprint Capacitor_SMD:C_0805_2012Metric_Pad1.18x1.45mm_HandSolder -> Capacitor_SMD:C_0402_1005Metric
- L301: value 10u -> 10n; footprint Inductor_SMD:L_0805_2012Metric_Pad1.05x1.20mm_HandSolder -> Capacitor_SMD:C_0603_1608Metric
- R301, R302, R303, R304, R305: footprint Resistor_SMD:R_0805_2012Metric_Pad1.20x1.40mm_HandSolder -> Resistor_SMD:R_0402_1005Metric
Connections:
- net CE_NRF: now also U301.2 (PF0); no longer U301.5 (PA0)
- net CSN_NRF: now also U301.3 (PF1); no longer U301.26 (PB3)
- net IMU_INT1: now also U301.26 (PB3); no longer U301.13 (PB0)
- net INT_BMS: now also U301.25 (PA15); no longer U301.6 (PA1)
- net IRQ_NRF: now also U301.5 (PA0); no longer U301.9 (PA4)
- net MOT_AIN2: now also U301.19 (PA9); no longer U301.21 (PA11)
- net MOT_BIN1: now also U301.22 (PA12); no longer U301.19 (PA9)
- net MOT_BIN2: now also U301.21 (PA11); no longer U301.22 (PA12)
- net OTG_HOST: now also U301.27 (PB4); no longer U301.7 (PA2)
- net TOF_INT1: now also U301.9 (PA4); no longer U301.2 (PF0)
- net TOF_INT2: now also U301.7 (PA2); no longer U301.3 (PF1)
- net XSHUT1: now also U301.13 (PB0); no longer U301.27 (PB4)
- net XSHUT2: now also U301.8 (PA3); no longer U301.28 (PB5)
- net ~{CE}_HOST: now also U301.28 (PB5); no longer U301.8 (PA3)
Changed lines of the file:
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@@
 	)
 	(no_connect
-		(at 149.86 119.38)
+		(at 149.86 83.82)
 	)
 	(no_connect
@@
 	(hierarchical_label "OTG_HOST"
 		(shape input)
-		(at 149.86 86.36 0)
+		(at 124.46 99.06 180)
 		(effects
 			(font
 				(size 1.27 1.27)
 			)
-			(justify left)
+			(justify right)
 		)
 	)
@@
 	(hierarchical_label "MOT_BIN2"
 		(shape bidirectional)
-		(at 149.86 111.76 0)
+		(at 149.86 109.22 0)
 		(effects
 			(font
@@
 	(hierarchical_label "CSN_NRF"
 		(shape output)
-		(at 124.46 96.52 180)
+		(at 124.46 88.9 180)
 		(effects
 			(font
@@
 	(hierarchical_label "INT_BMS"
 		(shape input)
-		(at 149.86 83.82 0)
+		(at 149.86 119.38 0)
 		(effects
 			(font
@@
 	(hierarchical_label "TOF_INT2"
 		(shape input)
-		(at 124.46 88.9 180)
+		(at 149.86 86.36 0)
 		(effects
 			(font
 				(size 1.27 1.27)
 			)
-			(justify right)
+			(justify left)
 		)
 	)
 	(hierarchical_label "MOT_AIN2"
 		(shape bidirectional)
-		(at 149.86 109.22 0)
+		(at 149.86 104.14 0)
 		(effects
 			(font
@@
 	(hierarchical_label "XSHUT2"
 		(shape output)
-		(at 124.46 101.6 180)
+		(at 149.86 88.9 0)
 		(effects
 			(font
 				(size 1.27 1.27)
 			)
-			(justify right)
+			(justify left)
 		)
 	)
@@
 	(hierarchical_label "~{CE}_HOST"
 		(shape input)
-		(at 149.86 88.9 0)
+		(at 124.46 101.6 180)
 		(effects
 			(font
 				(size 1.27 1.27)
 			)
-			(justify left)
+			(justify right)
 		)
 	)
 	(hierarchical_label "IMU_INT1"
 		(shape input)
-		(at 124.46 93.98 180)
+		(at 124.46 96.52 180)
 		(effects
 			(font
@@
 	(hierarchical_label "TOF_INT1"
 		(shape input)
-		(at 124.46 86.36 180)
+		(at 149.86 91.44 0)
 		(effects
 			(font
 				(size 1.27 1.27)
 			)
-			(justify right)
+			(justify left)
 		)
 	)
@@
 	(hierarchical_label "CE_NRF"
 		(shape output)
-		(at 149.86 81.28 0)
+		(at 124.46 86.36 180)
 		(effects
 			(font
 				(size 1.27 1.27)
 			)
-			(justify left)
+			(justify right)
 		)
 	)
 	(hierarchical_label "IRQ_NRF"
 		(shape input)
-		(at 149.86 91.44 0)
+		(at 149.86 81.28 0)
 		(effects
 			(font
@@
 	(hierarchical_label "XSHUT1"
 		(shape output)
-		(at 124.46 99.06 180)
+		(at 124.46 93.98 180)
 		(effects
 			(font
@@
 	(hierarchical_label "MOT_BIN1"
 		(shape bidirectional)
-		(at 149.86 104.14 0)
+		(at 149.86 111.76 0)
 		(effects
 			(font
@@
 			)
 		)
-		(property "Footprint" "Resistor_SMD:R_0805_2012Metric_Pad1.20x1.40mm_HandSolder"
+		(property "Footprint" "Resistor_SMD:R_0402_1005Metric"
 			(at 51.562 118.11 90)
 			(effects
@@
 			)
 		)
-		(property "Footprint" "Capacitor_SMD:C_0805_2012Metric_Pad1.18x1.45mm_HandSolder"
+		(property "Footprint" "Capacitor_SMD:C_0402_1005Metric"
 			(at 60.6552 45.72 0)
 			(effects
@@
 			)
 		)
-		(property "Footprint" "Resistor_SMD:R_0805_2012Metric_Pad1.20x1.40mm_HandSolder"
+		(property "Footprint" "Resistor_SMD:R_0402_1005Metric"
 			(at 43.942 118.11 90)
 			(effects
@@
 			)
 		)
-		(property "Footprint" "Resistor_SMD:R_0805_2012Metric_Pad1.20x1.40mm_HandSolder"
+		(property "Footprint" "Resistor_SMD:R_0402_1005Metric"
 			(at 85.852 74.93 90)
 			(effects
@@
 			)
 		)
-		(property "Value" "10u"
+		(property "Value" "10n"
 			(at 76.2 34.29 90)
 			(effects
@@
 			)
 		)
-		(property "Footprint" "Inductor_SMD:L_0805_2012Metric_Pad1.05x1.20mm_HandSolder"
+		(property "Footprint" "Capacitor_SMD:C_0603_1608Metric"
 			(at 76.2 36.83 0)
 			(effects
@@
 			)
 		)
-		(property "Footprint" "Capacitor_SMD:C_0805_2012Metric_Pad1.18x1.45mm_HandSolder"
+		(property "Footprint" "Capacitor_SMD:C_0402_1005Metric"
 			(at 97.4852 46.99 0)
 			(effects
@@
 			)
 		)
-		(property "Footprint" "Capacitor_SMD:C_0805_2012Metric_Pad1.18x1.45mm_HandSolder"
+		(property "Footprint" "Capacitor_SMD:C_0402_1005Metric"
 			(at 200.3552 57.15 0)
 			(effects
@@
 			)
 		)
-		(property "Footprint" "Capacitor_SMD:C_0805_2012Metric_Pad1.18x1.45mm_HandSolder"
+		(property "Footprint" "Capacitor_SMD:C_0402_1005Metric"
 			(at 35.2552 45.72 0)
 			(effects
@@
 			)
 		)
-		(property "Footprint" "Capacitor_SMD:C_0805_2012Metric_Pad1.18x1.45mm_HandSolder"
+		(property "Footprint" "Capacitor_SMD:C_0402_1005Metric"
 			(at 72.39 82.2452 0)
 			(effects
@@
 			)
 		)
-		(property "Footprint" "Resistor_SMD:R_0805_2012Metric_Pad1.20x1.40mm_HandSolder"
+		(property "Footprint" "Resistor_SMD:R_0402_1005Metric"
 			(at 59.182 118.11 90)
 			(effects
@@
 			)
 		)
-		(property "Footprint" "Resistor_SMD:R_0805_2012Metric_Pad1.20x1.40mm_HandSolder"
+		(property "Footprint" "Resistor_SMD:R_0402_1005Metric"
 			(at 93.472 123.19 90)
 			(effects
@@
 			)
 		)
-		(property "Footprint" "Capacitor_SMD:C_0805_2012Metric_Pad1.18x1.45mm_HandSolder"
+		(property "Footprint" "Capacitor_SMD:C_0402_1005Metric"
 			(at 47.9552 45.72 0)
 			(effects
@@
 			)
 		)
-		(property "Footprint" "Capacitor_SMD:C_0805_2012Metric_Pad1.18x1.45mm_HandSolder"
+		(property "Footprint" "Capacitor_SMD:C_0402_1005Metric"
 			(at 80.9752 46.99 0)
 			(effects
@@
 			)
 		)
-		(property "Footprint" "Capacitor_SMD:C_0805_2012Metric_Pad1.18x1.45mm_HandSolder"
+		(property "Footprint" "Capacitor_SMD:C_0402_1005Metric"
 			(at 234.6452 57.15 0)
 			(effects

Commit message: routage wip encore
Connections:
- net MOT_AIN1: now also U301.19 (PA9); no longer U301.18 (PA8)
- net MOT_AIN2: now also U301.20 (PA10); no longer U301.19 (PA9)
- net TOF_INT3: now also U301.18 (PA8); no longer U301.20 (PA10)
Changed lines of the file:
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@@
 	(hierarchical_label "MOT_AIN2"
 		(shape bidirectional)
-		(at 149.86 104.14 0)
+		(at 149.86 106.68 0)
 		(effects
 			(font
@@
 	(hierarchical_label "MOT_AIN1"
 		(shape bidirectional)
-		(at 149.86 101.6 0)
+		(at 149.86 104.14 0)
 		(effects
 			(font
@@
 	(hierarchical_label "TOF_INT3"
 		(shape input)
-		(at 149.86 106.68 0)
+		(at 149.86 101.6 0)
 		(effects
 			(font

Commit message: routage wip
Connections:
- net INT_BMS: now also U301.29 (PB6); no longer U301.25 (PA15)
- net XSHUT3: now also U301.25 (PA15); no longer U301.29 (PB6)
Changed lines of the file:
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@@
 	(hierarchical_label "INT_BMS"
 		(shape input)
-		(at 149.86 119.38 0)
+		(at 124.46 104.14 180)
 		(effects
 			(font
 				(size 1.27 1.27)
 			)
-			(justify left)
+			(justify right)
 		)
 	)
@@
 	(hierarchical_label "XSHUT3"
 		(shape output)
-		(at 124.46 104.14 180)
+		(at 149.86 119.38 0)
 		(effects
 			(font
 				(size 1.27 1.27)
 			)
-			(justify right)
+			(justify left)
 		)
 	)
