File: pcb/pcb_pcBOT/nrf.kicad_sch (KiCad schematic)
At the start: 0 parts

Commit message: ajout du module nrf + petites corrections
Parts:
- added C801: 10u, symbol Device:C
- added J802: nrF24l01_rf, symbol Connector_Generic:Conn_02x04_Odd_Even
Connections:
- new net: C801.1, J802.2 (Pin_2)
- new net CE_NRF: J802.3 (Pin_3)
- new net CSN_NRF: J802.4 (Pin_4)
- new net GND: J802.1 (Pin_1)
- new net IRQ_NRF: J802.8 (Pin_8)
- new net MISO_NRF: J802.7 (Pin_7)
- new net MOSI_NRF: J802.6 (Pin_6)
- new net SCK_NRF: J802.5 (Pin_5)
- new net VDD: C801.2
Other:
- note added: "module de communication"
- company: (none) -> ENSEA G5
- title: (none) -> nrF_PcBot

Commit message: complement tof et connections, mise a jour du firmware
Other:
- note added: "communication module"
- note removed: "module de communication"
Changed lines of the file:
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@@
 		(company "ENSEA G5")
 	)
-	(text "module de communication \n"
+	(text "communication module\n"
 		(exclude_from_sim no)
-		(at 146.812 103.378 0)
+		(at 145.034 103.378 0)
 		(effects
 			(font

Commit message: Ajout empreintes (incomplet) + test erc correct
Parts:
- C801: footprint (none) -> Capacitor_SMD:C_0805_2012Metric_Pad1.18x1.45mm_HandSolder
- J802: footprint (none) -> Connector_PinHeader_2.54mm:PinHeader_2x04_P2.54mm_Vertical
Changed lines of the file:
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@@
 			)
 		)
-		(property "Footprint" ""
+		(property "Footprint" "Connector_PinHeader_2.54mm:PinHeader_2x04_P2.54mm_Vertical"
 			(at 144.78 88.9 0)
 			(effects
@@
 			)
 		)
-		(property "Footprint" ""
+		(property "Footprint" "Capacitor_SMD:C_0805_2012Metric_Pad1.18x1.45mm_HandSolder"
 			(at 175.26 85.3948 0)
 			(effects

Commit message: Revert "Ajout empreintes (incomplet) + test erc correct"
This reverts commit 267ed5519d67c336b99c9c80b0ac2067182b82a3.
Parts:
- C801: footprint Capacitor_SMD:C_0805_2012Metric_Pad1.18x1.45mm_HandSolder -> (none)
- J802: footprint Connector_PinHeader_2.54mm:PinHeader_2x04_P2.54mm_Vertical -> (none)
Changed lines of the file:
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@@
 			)
 		)
-		(property "Footprint" "Connector_PinHeader_2.54mm:PinHeader_2x04_P2.54mm_Vertical"
+		(property "Footprint" ""
 			(at 144.78 88.9 0)
 			(effects
@@
 			)
 		)
-		(property "Footprint" "Capacitor_SMD:C_0805_2012Metric_Pad1.18x1.45mm_HandSolder"
+		(property "Footprint" ""
 			(at 175.26 85.3948 0)
 			(effects
