File: pcb/pcb_pcBOT/nrf.kicad_sch (KiCad schematic)
At the start: 2 parts, among them J802 nrF24l01_rf

Commit message: rouatage + firmware wip
Parts:
- C801: footprint Capacitor_SMD:C_0805_2012Metric_Pad1.18x1.45mm_HandSolder -> Capacitor_SMD:C_0603_1608Metric
Changed lines of the file:
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@@
 			)
 		)
-		(property "Footprint" "Capacitor_SMD:C_0805_2012Metric_Pad1.18x1.45mm_HandSolder"
+		(property "Footprint" "Capacitor_SMD:C_0603_1608Metric"
 			(at 175.26 85.3948 0)
 			(effects
