File: pcb/pcb_pcBOT/pcb_pcBOT.kicad_pcb (KiCad board)
At the start: 2 copper layers, 66 parts, among them J201 Lipo, J202 USB_C_Receptacle_USB2.0_16P, J302 Conn_ST_STDC14, J501 TOF1, J502 TOF2, J503 TOF3, J802 nrF24l01_rf, SW201 ~{QON}_BUTTON, SW301 Reset_Button, U201 BQ25896RTW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

Commit message: début routage premier jet
Parts:
- added REF**: MountingHole_2.1mm, MountingHole:MountingHole_2.1mm, F.Cu at (127.3, 71.1)
- added REF**: MountingHole_2.1mm, MountingHole:MountingHole_2.1mm, F.Cu at (181.4, 71.1)
- added REF**: MountingHole_2.1mm, MountingHole:MountingHole_2.1mm, F.Cu at (182.1, 115.6)
- added REF**: MountingHole_2.1mm, MountingHole:MountingHole_2.1mm, F.Cu at (127.8, 115.3)
- moved C307 50.3 mm to (158.8, 105.4), turned to -90 degrees
- moved C309 42.6 mm to (151.6, 105.4), turned to 90 degrees
- moved C303 42.1 mm to (151.9, 88.7), turned to 90 degrees
- moved C302 40.7 mm to (148.8, 88.7), turned to 90 degrees
- moved SW201 40.5 mm to (183.3, 100.7), turned to -90 degrees
- moved C301 39.7 mm to (145.8, 88.7), turned to 90 degrees
- moved R504 38.5 mm to (139.7, 75.2), turned to 135 degrees
- moved C208 38.5 mm to (175.7, 104.0), turned to 90 degrees
- moved Moteur701 37.4 mm to (163.1, 71.6)
- moved R502 36.7 mm to (141.2, 73.7), turned to 135 degrees
- moved R303 36.4 mm to (142.3, 110.5), turned to 180 degrees
- moved R206 35.2 mm to (177.3, 87.6)
- moved U303 34.7 mm to (155.1, 105.6), turned to 180 degrees
- moved R-IPROPI_A701 33.7 mm to (174.5, 108.5), turned to 90 degrees
- moved R302 33.6 mm to (149.3, 92.5)
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Other:
- board outline added: 60.7 x 50.5 mm

Commit message: routage wip
Parts:
- C301, C302, C303, C305, C306, JP201, JP202, JP203, R-IPROPI_A701, R-IPROPI_B701, R207, R208, R301: moved to B.Cu
- moved JP201 53.3 mm to (201.7, 93.0), turned to 180 degrees
- moved JP202 48.6 mm to (201.7, 95.7), turned to 180 degrees
- moved JP203 47.7 mm to (201.6, 90.3)
- moved Moteur701 46.7 mm to (148.8, 116.1), turned to 180 degrees
- moved J802 46.1 mm to (154.2, 69.8), turned to -90 degrees
- moved SW301 37.0 mm to (167.2, 112.1), turned to 0 degrees
- moved C304 36.0 mm to (164.7, 114.8), turned to 90 degrees
- moved C801 34.5 mm to (154.1, 75.2), turned to 0 degrees
- moved R209 24.6 mm to (171.0, 94.3), turned to -90 degrees
- moved R210 21.4 mm to (173.0, 94.3), turned to -90 degrees
- moved C701 16.8 mm to (158.7, 105.3)
- moved Cbulk701 16.7 mm to (158.7, 107.6)
- moved U701 16.0 mm to (152.5, 107.5), turned to 90 degrees
- moved C201 15.7 mm to (167.4, 89.4), turned to -90 degrees
- moved R208 15.1 mm to (171.5, 79.7), turned to 0 degrees
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Connections:
- U301 pad 13: /centrale imu/IMU_INT1 -> /capteur tof/TOF_INT1
- U301 pad 18: /driver_motor/PWM -> /driver_motor/MOT_AIN1
- U301 pad 19: /driver_motor/PWM -> /driver_motor/MOT_BIN1
- U301 pad 2: /capteur tof/TOF_INT1 -> /centrale imu/IMU_INT1
- U301 pad 21: /driver_motor/PWM -> /driver_motor/MOT_AIN2
- U301 pad 22: /driver_motor/PWM -> /driver_motor/MOT_BIN2
- U301 pad 25: unconnected-(U301-PA15-Pad25) -> /bms/INT_BMS
- U301 pad 6: /bms/INT_BMS -> unconnected-(U301-PA1-Pad6)
- U701 pad 10: /driver_motor/PWM -> /driver_motor/MOT_BIN2
- U701 pad 15: /driver_motor/PWM -> /driver_motor/MOT_AIN2
- U701 pad 16: /driver_motor/PWM -> /driver_motor/MOT_AIN1
- U701 pad 2: Net-(Moteur701-Pin_1) -> Net-(Moteur701-Pin_2)
- U701 pad 4: Net-(Moteur701-Pin_2) -> Net-(Moteur701-Pin_1)
- U701 pad 9: /driver_motor/PWM -> /driver_motor/MOT_BIN1
Routing:
- net VDD: track 0.00 -> 47.4 mm
- net /capteur tof/TOF_INT3: track 0.00 -> 3.97 mm
- net /capteur tof/TOF_INT2: track 0.00 -> 3.94 mm
- net /capteur tof/XSHUT2: track 0.00 -> 3.50 mm
- net /capteur tof/XSHUT3: track 0.00 -> 2.91 mm
Other:
- copper layers 2 -> 4

Commit message: rouatage + firmware wip
Parts:
- removed REF** (x4): MountingHole_2.1mm, MountingHole:MountingHole_2.1mm
- added H101: MountingHole_Pad, MountingHole:MountingHole_3.2mm_M3_Pad_Via, F.Cu at (130.0, 70.0)
- added H102: MountingHole_Pad, MountingHole:MountingHole_3.2mm_M3_Pad_Via, F.Cu at (190.0, 70.0)
- added H103: MountingHole_Pad, MountingHole:MountingHole_3.2mm_M3_Pad_Via, F.Cu at (190.0, 120.0)
- added H104: MountingHole_Pad, MountingHole:MountingHole_3.2mm_M3_Pad_Via, F.Cu at (130.0, 120.0)
- C201, C203, C208, C304, C307, C309, C601, C602: footprint Capacitor_SMD:C_0805_2012Metric_Pad1.18x1.45mm_HandSolder -> Capacitor_SMD:C_0402_1005Metric
- C202, C204, C205, C206, C207, C801: footprint Capacitor_SMD:C_0805_2012Metric_Pad1.18x1.45mm_HandSolder -> Capacitor_SMD:C_0603_1608Metric
- C301, C302, C303, C305, C306: footprint Capacitor_SMD:C_0805_2012Metric_Pad1.18x1.45mm_HandSolder -> Capacitor_SMD:C_0402_1005Metric; moved to F.Cu
- C701: value 100nF -> 100n; footprint Capacitor_SMD:C_0805_2012Metric_Pad1.18x1.45mm_HandSolder -> Capacitor_SMD:C_0402_1005Metric
- Cbulk701: value 10µF -> 10u; footprint Capacitor_SMD:C_0805_2012Metric_Pad1.18x1.45mm_HandSolder -> Capacitor_SMD:C_0603_1608Metric
- D201, D202: footprint LED_SMD:LED_0603_1608Metric_Pad1.05x0.95mm_HandSolder -> Capacitor_SMD:C_0402_1005Metric
- L201: footprint Inductor_SMD:L_0805_2012Metric_Pad1.05x1.20mm_HandSolder -> Inductor_SMD:L_1008_2520Metric
- L301: value 10u -> 10n; footprint Inductor_SMD:L_0805_2012Metric_Pad1.05x1.20mm_HandSolder -> Capacitor_SMD:C_0603_1608Metric
- R-IPROPI_A701, R-IPROPI_B701: value 16.5 kΩ -> 16k5; footprint Resistor_SMD:R_0805_2012Metric_Pad1.20x1.40mm_HandSolder -> Resistor_SMD:R_0402_1005Metric
- R202, R204, R206, R207, R209, R210, R302, R303, R304, R305, R501, R502, R503, R504, R505, R506, R601: footprint Resistor_SMD:R_0805_2012Metric_Pad1.20x1.40mm_HandSolder -> Resistor_SMD:R_0402_1005Metric
- R208, R301: footprint Resistor_SMD:R_0805_2012Metric_Pad1.20x1.40mm_HandSolder -> Resistor_SMD:R_0402_1005Metric; moved to F.Cu
- Rvmcu701: value 10 kΩ -> 10k; footprint Resistor_SMD:R_0805_2012Metric_Pad1.20x1.40mm_HandSolder -> Resistor_SMD:R_0402_1005Metric
- moved JP202 31.9 mm to (170.3, 90.0)
- moved JP201 31.9 mm to (170.3, 87.4)
- moved JP203 31.4 mm to (170.3, 92.5)
- moved SW201 27.0 mm to (192.3, 75.2)
- moved C208 25.9 mm to (191.8, 83.8), turned to 180 degrees
- moved R209 21.3 mm to (190.3, 85.5), turned to 0 degrees
- moved C201 16.9 mm to (183.6, 94.2)
- moved R301 15.4 mm to (158.8, 91.7), turned to 180 degrees
- moved R501 14.0 mm to (128.9, 100.2), turned to 90 degrees
- moved R210 10.2 mm to (183.1, 92.6), turned to 180 degrees
- moved J201 9.94 mm to (178.6, 68.4), turned to 0 degrees
- moved J202 9.93 mm to (190.3, 91.3)
- moved R506 9.62 mm to (128.2, 97.5)
- moved R202 9.55 mm to (175.9, 100.7)
- moved R204 9.55 mm to (173.9, 100.7)
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Connections:
- net Net-(JP201-B) renamed /bms/VBUS_BQ25
- U301 pad 13: /capteur tof/TOF_INT1 -> /capteur tof/XSHUT1
- U301 pad 19: /driver_motor/MOT_BIN1 -> /driver_motor/MOT_AIN2
- U301 pad 2: /centrale imu/IMU_INT1 -> /SPI_BUS.CE_NRF
- U301 pad 21: /driver_motor/MOT_AIN2 -> /driver_motor/MOT_BIN2
- U301 pad 22: /driver_motor/MOT_BIN2 -> /driver_motor/MOT_BIN1
- U301 pad 26: /SPI_BUS.CSN_NRF -> /centrale imu/IMU_INT1
- U301 pad 27: /capteur tof/XSHUT1 -> /bms/OTG_HOST
- U301 pad 28: /capteur tof/XSHUT2 -> /bms/~{CE}_HOST
- U301 pad 3: /capteur tof/TOF_INT2 -> /SPI_BUS.CSN_NRF
- U301 pad 5: /SPI_BUS.CE_NRF -> /nrf24l01/IRQ_NRF
- U301 pad 7: /bms/OTG_HOST -> /capteur tof/TOF_INT2
- U301 pad 8: /bms/~{CE}_HOST -> /capteur tof/XSHUT2
- U301 pad 9: /nrf24l01/IRQ_NRF -> /capteur tof/TOF_INT1
Routing:
- net VDD: track 47.4 -> 0.00 mm, vias 0 -> 1
- net /capteur tof/TOF_INT2: track 3.94 -> 24.8 mm
- net /capteur tof/XSHUT1: track 0.00 -> 20.3 mm
- net /capteur tof/XSHUT2: track 3.50 -> 23.8 mm
- net /capteur tof/TOF_INT1: track 0.00 -> 18.1 mm
- net /stm32/NRST: track 0.00 -> 9.65 mm
- net /driver_motor/MOT_BIN1: track 0.00 -> 9.11 mm
- net /driver_motor/MOT_BIN2: track 0.00 -> 8.62 mm
- net /bms/~{QON}: track 0.00 -> 8.55 mm
- net /driver_motor/MOT_AIN1: track 0.00 -> 7.80 mm
- net /driver_motor/MOT_AIN2: track 0.00 -> 7.74 mm
- net VDDA: track 0.00 -> 5.49 mm
- net Net-(J802-Pin_2): track 0.00 -> 3.30 mm
- net /bms/PMID: track 0.00 -> 3.28 mm
- net GND: track 0.00 -> 3.20 mm, vias 0 -> 5
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- added copper zone on In2.Cu, net +5V
- added copper zone on F.Cu, net /bms/VBUS_BQ25
- added copper zone on In1.Cu, net GND
- added copper zone on F.Cu, net Net-(Moteur702-Pin_2)
- added copper zone on In2.Cu, net VDD
Other:
- board size 60.7 x 50.5 mm -> 68 x 58 mm

Commit message: routage wip
Parts:
- moved R305 39.5 mm to (178.0, 85.0)
- moved C602 28.1 mm to (177.0, 96.7), turned to 90 degrees
- moved C601 27.3 mm to (174.7, 98.7), turned to 0 degrees
- moved U601 24.5 mm to (174.7, 96.7), turned to 0 degrees
- moved R601 20.9 mm to (172.4, 96.4), turned to 90 degrees
- moved R301 10.8 mm to (151.1, 84.2), turned to -90 degrees
- moved D202 9.11 mm to (171.1, 95.5)
- moved D201 8.83 mm to (169.6, 95.4)
- moved SW201 7.91 mm to (187.8, 81.7), turned to 90 degrees
- moved R204 7.88 mm to (171.2, 93.4), turned to 90 degrees
- moved R202 6.89 mm to (175.2, 93.9), turned to 90 degrees
- moved Moteur701 5.40 mm to (150.8, 120.5)
- moved Moteur702 5.40 mm to (157.8, 120.5)
- moved C208 3.47 mm to (188.3, 83.8), turned to 0 degrees
- moved C304 1.79 mm to (169.7, 118.0)
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Routing:
- net /centrale imu/IMU_INT1: track 0.00 -> 19.7 mm
- net /bms/~{QON}: track 8.55 -> 24.0 mm
- net /bms/~{PG}: track 0.00 -> 7.39 mm
- net /bms/INT_BMS: track 0.00 -> 4.79 mm
- net /stm32/NRST: track 9.65 -> 12.9 mm
- net I: track 0.00 -> 2.90 mm
- net /capteur tof/TOF_INT1: track 18.1 -> 20.5 mm
- net Net-(D202-K): track 0.00 -> 1.11 mm
- added copper zone on F.Cu, net Net-(Moteur701-Pin_1)
- added copper zone on F.Cu, net Net-(Moteur701-Pin_2)
- added copper zone on F.Cu, net Net-(Moteur702-Pin_1)

Commit message: routage wip encore
Parts:
- R-IPROPI_A701, R-IPROPI_B701: moved to F.Cu
- moved J302 41.5 mm to (189.6, 105.4), turned to 180 degrees
- moved R-IPROPI_A701 13.0 mm to (153.2, 101.5), turned to 135 degrees
- moved C601 11.1 mm to (180.3, 108.2)
- moved C602 11.1 mm to (182.6, 106.3)
- moved R601 11.1 mm to (178.0, 106.0)
- moved U601 11.1 mm to (180.3, 106.2)
- moved R209 9.26 mm to (182.1, 89.6), turned to 180 degrees
- moved C801 7.27 mm to (163.7, 73.2)
- moved J802 6.90 mm to (162.8, 68.1)
- moved C701 5.92 mm to (154.9, 103.0)
- moved R301 5.15 mm to (151.2, 79.0)
- moved R303 4.78 mm to (140.6, 104.5)
- moved R304 4.78 mm to (140.7, 103.4)
- moved D201 4.34 mm to (173.6, 97.0)
- moved L201 2.30 mm to (167.1, 80.2)
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Connections:
- net /SPI_BUS.CE_NRF renamed /nrf24l01/CE_NRF
- net /SPI_BUS.CSN_NRF renamed /nrf24l01/CSN_NRF
- U301 pad 18: /driver_motor/MOT_AIN1 -> /capteur tof/TOF_INT3
- U301 pad 19: /driver_motor/MOT_AIN2 -> /driver_motor/MOT_AIN1
- U301 pad 20: /capteur tof/TOF_INT3 -> /driver_motor/MOT_AIN2
Routing:
- net /stm32/T_SWDIO: track 0.00 -> 45.1 mm
- net /SPI_BUS.MOSI_NRF: track 0.00 -> 43.9 mm, vias 0 -> 2
- net /stm32/T_SWCLK: track 0.00 -> 41.2 mm
- net /SPI_BUS.SCK_NRF: track 0.00 -> 33.8 mm, vias 0 -> 2
- net /SPI_BUS.MISO_NRF: track 0.00 -> 33.3 mm, vias 0 -> 2
- net /nrf24l01/CE_NRF: track 0.00 -> 24.9 mm
- net /capteur tof/TOF_INT3: track 2.43 -> 26.6 mm
- net /nrf24l01/CSN_NRF: track 0.00 -> 21.7 mm
- net /nrf24l01/IRQ_NRF: track 0.00 -> 20.8 mm
- net /bms/BAT: track 0.00 -> 16.3 mm
- net VBUS: track 3.07 -> 14.8 mm, vias 0 -> 1
- net /bms/STAT: track 0.00 -> 9.69 mm
- net /centrale imu/IMU_INT1: track 19.7 -> 29.3 mm
- net /stm32/NRST: track 12.9 -> 18.1 mm
- net Net-(J202-CC2): track 0.00 -> 4.10 mm
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- added copper zone on F.Cu, net /bms/PMID
- added copper zone on F.Cu, net /bms/REGN

Commit message: routage wip
Parts:
- moved R-B701 11.5 mm to (156.7, 101.8), turned to 90 degrees
- moved R304 7.21 mm to (137.8, 110.0), turned to -135 degrees
- moved R303 6.60 mm to (138.5, 110.8), turned to -135 degrees
- moved U601 5.59 mm to (175.4, 103.5)
- moved C601 5.59 mm to (175.4, 105.5)
- moved R601 5.59 mm to (173.2, 103.3)
- moved C602 5.51 mm to (177.7, 103.8)
- moved C309 4.94 mm to (159.6, 101.8)
- moved R301 4.80 mm to (151.2, 83.8)
- moved U303 4.66 mm to (162.2, 101.7)
- moved C307 4.00 mm to (164.8, 101.2)
- moved R305 2.32 mm to (176.8, 87.0)
- moved R-IPROPI_A701 1.70 mm to (152.0, 100.2)
- moved R208 1.58 mm to (176.4, 82.6)
- moved R206 1.58 mm to (176.4, 83.6)
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- renumbered R-IPROPI_B701 to R-B701
Connections:
- U201 pad 5: /I2C_BUS.I2C_SCL -> /I2C_BUS.I2C_SDA
- U201 pad 6: /I2C_BUS.I2C_SDA -> /I2C_BUS.I2C_SCL
- U301 pad 25: /bms/INT_BMS -> /capteur tof/XSHUT3
- U301 pad 29: /capteur tof/XSHUT3 -> /bms/INT_BMS
Routing:
- net /I2C_BUS.I2C_SDA: track 0.00 -> 132.0 mm, vias 0 -> 6
- net /I2C_BUS.I2C_SCL: track 4.08 -> 125.8 mm, vias 0 -> 6
- net /stm32/NRST: track 18.1 -> 135.8 mm, vias 0 -> 5
- net /bms/~{CE}_HOST: track 0.00 -> 48.8 mm, vias 0 -> 2
- net /bms/SYS: track 0.14 -> 36.6 mm, vias 0 -> 1
- net /bms/INT_BMS: track 4.79 -> 38.2 mm, vias 0 -> 2
- net /capteur tof/XSHUT3: track 2.42 -> 33.6 mm, vias 0 -> 2
- net /bms/OTG_HOST: track 0.00 -> 28.1 mm, vias 0 -> 2
- net +5V: track 0.00 -> 17.5 mm, vias 3 -> 6
- net VBUS: track 14.8 -> 29.5 mm
- net /bms/REGN: track 0.00 -> 10.5 mm, vias 0 -> 1
- net GND: track 3.20 -> 10.5 mm, vias 25 -> 37
- net VDD: track 0.00 -> 6.87 mm, vias 1 -> 21
- net /bms/TS: track 1.77 -> 8.27 mm, vias 0 -> 1
- net /centrale imu/IMU_INT1: track 29.3 -> 23.4 mm
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- added copper zone on F.Cu, net /bms/ILIM
- added copper zone on F.Cu, net /bms/SYS
- added copper zone on F.Cu, net /bms/TS

Commit message: fin du routage
Parts:
- moved JP203 14.7 mm to (164.1, 79.2), turned to 180 degrees
- moved JP201 12.2 mm to (182.5, 87.5)
- moved R209 10.6 mm to (191.8, 85.2), turned to 0 degrees
- moved JP202 9.85 mm to (171.3, 99.8)
- moved C309 9.44 mm to (166.1, 108.6), turned to 180 degrees
- moved R210 8.56 mm to (190.2, 97.2), turned to 0 degrees
- moved U303 5.78 mm to (166.0, 106.0), turned to -90 degrees
- moved C307 2.26 mm to (165.6, 103.3), turned to 0 degrees
- moved R-B701 0.78 mm to (155.9, 102.2)
- moved C701 0.69 mm to (154.8, 102.2)
- moved R305 0.67 mm to (176.2, 86.5), turned to -90 degrees
- moved R601 0.56 mm to (172.7, 103.0)
- moved D201 0.16 mm to (173.5, 96.8)
- moved R202 0.10 mm to (173.5, 94.9)
Routing:
- net /stm32/NRST: track 135.8 -> 83.2 mm, vias 5 -> 2
- net +5V: track 17.5 -> 2.22 mm
- net VBUS: track 29.5 -> 14.2 mm, vias 1 -> 5
- net Net-(JP202-B): track 0.00 -> 14.2 mm, vias 0 -> 1
- net GND: track 10.5 -> 20.0 mm, vias 37 -> 60
- net /bms/SYS: track 36.6 -> 30.2 mm
- net /I2C_BUS.I2C_SDA: track 132.0 -> 126.9 mm
- net /bms/SW: track 4.38 -> 0.10 mm
- net /bms/BAT: track 18.6 -> 14.5 mm
- net Net-(J202-CC1): track 3.10 -> 6.28 mm
- net Net-(J202-CC2): track 4.10 -> 6.96 mm
- net /I2C_BUS.I2C_SCL: track 125.8 -> 123.1 mm
- net VDD: track 6.87 -> 8.29 mm, vias 21 -> 24
- net Net-(U601-SDO/SA0): track 1.22 -> 2.37 mm
- net /nrf24l01/IRQ_NRF: track 21.4 -> 20.3 mm
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- added copper zone on F.Cu, net /bms/BAT
- added copper zone on F.Cu, net /bms/SW
- added copper zone on In2.Cu, net /bms/VBUS_BQ25
- added copper zone on B.Cu, net GND
- added copper zone on F.Cu, net GND
- added copper zone on In2.Cu, net VBUS

Commit message: pcb v1 fini fichier envoyé à jlc
Parts:
- added G***: LOGO, LOGO, F.Cu at (138.8, 79.0)
- added G***: LOGO, LOGO, F.Cu at (172.8, 111.7)
Routing:
- net /stm32/T_SWCLK: track 40.4 -> 39.4 mm
- net /bms/~{CE}_HOST: track 48.6 -> 49.5 mm
- net GND: vias 60 -> 64
Other:
- board text added: "PcBot G5"
