File: pcb/pcb_pcBOT/pcb_pcBOT.kicad_pcb (KiCad board)
At the start: 4 copper layers, 68 x 58 mm, 72 parts, among them J201 Lipo, J202 USB_C_Receptacle_USB2.0_16P, J302 Conn_ST_STDC14, J501 TOF1, J502 TOF2, J503 TOF3, J802 nrF24l01_rf, SW201 ~{QON}_BUTTON, SW301 Reset_Button, U201 BQ25896RTW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

Commit message: tof codes
Parts:
- removed G*** (x2): LOGO, LOGO
Routing:
- net /stm32/T_SWCLK: track 39.4 -> 40.4 mm
- net /bms/~{CE}_HOST: track 49.5 -> 48.6 mm
- net GND: vias 64 -> 60
Other:
- board text removed: "PcBot G5"
